File: drums.sch (EAGLE design)
At the start: 294 parts, among them IC1 4051N, IC2 4584N, IC3 7812T, IC5 OPA2134P, IC6 OPA4130P, IC7 LM2574HVN-5.0, IC8 74LS595N, IC9 OPA4130P, J2 UBBS-4R-D14-4D

Commit message: added toms
Parts:
- added C67, C85: 33u, dan:CPOL-USE2-5
- added C68: 4.7n, dan:C-US050-025X075
- added C69, C70: 27n, dan:C-US050-025X075
- added C71, C78: 47u, dan:CPOL-USE2-5
- added C72: .47u, dan:C-US050-025X075
- added C73: 3.9n, dan:C-US050-025X075
- added C74, C75, C81: 18n, dan:C-US050-025X075
- added C76: 68n, dan:C-US050-025X075
- added C77, C79: 47n, dan:C-US050-025X075
- added C80: 39n, dan:C-US050-025X075
- added C82: 10n, dan:C-US050-025X075
- added C83, C84: 1u, dan:CPOL-USE2-5
- added D17, D18: 1N4148DO35-7, dan:1N4148DO35-7
- added HATSLEVEL1: 500k, dan:US-EVUF2J
- added HTOMTUN, LTOMTUN: 1k, dan:US-EVUF2J
- added IC10: OPA2134P, dan:OPA2134P
- added LTOMDEC: 1M, dan:US-EVUF2J
- added R138, R151, R153, R166, R178: 100k, dan:R-US_0207/2V
- added R139, R182, R183: 15k, dan:R-US_0207/2V
- added R140, R157: 1k, dan:R-US_0207/2V
- added R141, R158, R174, R176, R177, R179: 4.7k, dan:R-US_0207/2V
- added R142, R144, R145, R146, R147, R154, R159, R161, R162, R163, R164, R175, R180: 10k, dan:R-US_0207/2V
- added R143, R160, R181: 22k, dan:R-US_0207/2V
- added R148, R165, R184, R186: 47k, dan:R-US_0207/2V
- added R149, R167: 2.2M, dan:R-US_0207/2V
- added R150, R152, R168: 100, dan:R-US_0207/2V
- added R155, R169: 680k, dan:R-US_0207/2V
- added R156: 72k, dan:R-US_0207/2V
- added R170: 39k, dan:R-US_0207/2V
- added R171: 2.2k, dan:R-US_0207/2V
- added R172: 1M, dan:R-US_0207/2V
- added R173, R185: 33k, dan:R-US_0207/2V
- added TOMLEV: 10k, dan:US-EVUF2J
- added U$23, U$27, U$28: 2N3906_, dan:2N3906_
- added U$24, U$25, U$26, U$29, U$30, U$31, U$32: 2N3904_, dan:2N3904_
- BASSTONE: value US-EVUF2J -> 10k
- BASSTUNE: value US-EVUF2J -> 250k
Connections:
- net N$147 renamed T8B
- net N$148 renamed T10B
- removed net N$135: JP8.9
- removed net N$139: JP7.6
- removed net N$140: JP7.8
- removed net N$141: JP7.10
- removed net N$39: JP7.9
- removed net T5B: JP8.3, R115.2
- new net CHATLEV2A: HATSLEVEL1.A, JP7.7
- new net CHATLEV2B: C67.-, JP8.7
- new net CHATLEVA: HATSLEVEL1.E, HATSLEVEL1.S, JP7.6
- new net CHATLEVB: IC9C.OUT, JP8.6, R138.1
- new net HTOMTUNA: HTOMTUN.E, HTOMTUN.S
- new net HTOMTUNB: R168.2, U$30.C
- new net LTOMDEC2A: LTOMDEC.E
- new net LTOMDEC2B: C85.+
- new net LTOMDECA: LTOMDEC.A, LTOMDEC.S
- new net LTOMDECB: IC10A.OUT, R184.1, R186.2
- new net LTOMTUNA: LTOMTUN.E, LTOMTUN.S
- new net LTOMTUNB: R150.2, U$25.C
- new net N$132: C68.2, IC9D.+IN, R148.2
- new net N$137: C70.2, IC9D.OUT, R149.1, R183.1, R185.2
- new net N$138: C69.2, C70.1, R150.1, R186.1
- new net N$144: C71.+, R152.2, R153.1, U$27.E
- new net N$145: C76.1, R171.1, R172.2
- new net N$157: C72.1, R155.2, R169.1, U$27.C
- new net N$165: R154.2, U$27.B
- new net N$167: R155.1, R156.2, U$25.B
- new net N$174: C77.2, R172.1, R173.2
- new net N$175: D18.A, R164.2, R166.2, U$28.C
- new net N$182: R158.1, R159.2, U$28.B
- new net N$186: R158.2, R162.1, R163.1, U$28.E
- new net N$190: R159.1, U$29.C
- new net N$191: R160.1, R161.1, U$29.B
- new net N$192: C73.1, R157.2, R164.1
- new net N$193: C73.2, IC10B.+IN, R165.2
- new net N$194: R151.1, R166.1, U$26.B
- new net N$195: D17.C, D18.C, R171.2
- new net N$196: R173.1, U$31.B
- new net N$197: C74.1, IC10B.-IN, R167.2
- new net N$198: C75.2, IC10B.OUT, R167.1, R182.1
- new net N$199: C74.2, C75.1, R168.1
- new net N$2: C67.+, IC9C.-IN, R136.1, R138.2
- new net N$201: R169.2, R170.2, U$30.B
- new net N$202: C79.1, R174.2, U$31.C
- new net N$203: C78.+, R174.1, R175.2
- new net N$204: C77.1, R179.1, R180.2
- new net N$205: C81.2, R181.1, U$32.B
- new net N$206: C79.2, R176.1, R177.1
- new net N$207: C80.1, U$32.E
- new net N$208: C82.2, R177.2, R178.1
- new net N$209: C85.-, IC10A.-IN, R184.2, R185.1
- new net N$210: C84.+, R182.2
- new net N$211: C83.+, R183.2
- new net N$215: TOMLEV.S
- new net N$216: U$1.23/A9/T/PWM
- new net N$218: U$1.22/A8/T/PWM
- new net N$32: R139.1
- new net N$35: D17.A, R147.2, R151.2, U$23.C
- new net N$36: R141.1, R142.2, U$23.B
- new net N$37: R141.2, R145.1, R146.1, U$23.E
- new net N$48: R143.1, R144.1, U$24.B
- new net N$50: C68.1, R140.2, R147.1
- new net T10: JP7.10, U$1.21/A7/PWM
- new net T9: JP7.9, U$1.20/A6/PWM
- new net T9B: JP8.3, JP8.9, R115.2, R143.2, R160.2
- new net TOMSLEVA: TOMLEV.A
- new net TOMSLEVB: C83.-, C84.-, R178.2
- net +12V: now also IC10P.V-, R145.2, R152.1, R162.2, R175.1, U$32.C
- net -12V: now also IC10P.V+
- net GND: now also C71.-, C72.2, C76.2, C78.-, C81.1, C82.1, HTOMTUN.A, IC10A.+IN, IC9C.+IN, LTOMTUN.A, R140.1, R144.2, R148.1, R156.1, R157.1, R161.2, R165.1, R170.1, R176.2, R179.2, TOMLEV.E, U$24.E, U$25.E, U$26.E, U$29.E, U$30.E, U$31.E
- net N$134: now also C69.1, IC9D.-IN, R149.2; no longer JP8.7
- net N$146: now also R153.2, R154.1, U$26.C; no longer JP8.6
- net N$177: now also R139.2
- net N$189: no longer R136.1
- net N$38: now also R142.1, U$24.C; no longer JP7.7
- net T7B: now also R146.2, R163.2
- net T8: now also JP7.8
- net WNOISE: now also C80.2, R180.1, R181.2
Other:
- note added: "check this, might be in series"
- moved on the sheet: C49, C50, C51, C52, C53, C54, C55, C56, C57, C58, C59, C60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
